File: Hardware/DataAcq-EnvironmentBoard.kicad_pcb (KiCad board)
At the start: 2 copper layers, 53.9 x 59 mm, 33 parts, among them J2 CAN Output, J3 CAN Input, J6 Breakout Connector, U1 SHT45, U2 FS3000-1005, U3 LMT87DCK, U4 Daughterboard Connector

Commit message: new ptc & footprints
Parts:
- removed C1, C2, C3, C5, C6: 0.1uF, Capacitor_SMD:C_0805_2012Metric
- removed C4, C7: 1uF, Capacitor_SMD:C_0805_2012Metric
- removed D1: 12V, LED_SMD:LED_0805_2012Metric
- removed D2: 3.3V, LED_SMD:LED_0805_2012Metric
- removed D3, D4, D5, D6: ESD9B, Diode_SMD:D_SOD-923
- removed F1, F2: 250mA, Fuse:Fuse_0603_1608Metric
- removed J2: CAN Output, UTSVT_Connectors:Molex_MicroFit3.0_1x4xP3.00mm_PolarizingPeg_Vertical
- removed J3: CAN Input, UTSVT_Connectors:Molex_MicroFit3.0_1x4xP3.00mm_PolarizingPeg_Vertical
- removed J6: Breakout Connector, Connector_Molex:Molex_Nano-Fit_105310-xx10_2x05_P2.50mm_Vertical
- removed LOGO1: Arrow, images:arrow
- removed LOGO2: Dr. Hallock, UTSVT_Special:Hallock_Image_Tiny
- removed LOGO3: UTSVT Logo, UTSVT_Special:UTSVT_Logo_Symbol
- removed LOGO4: Wolf, images:wolf
- removed R1: 1k, Resistor_SMD:R_0805_2012Metric
- removed R2: 22.1k, Resistor_SMD:R_0805_2012Metric
- removed R3: 2.2k, Resistor_SMD:R_0805_2012Metric
- removed TP1, TP2, TP4, TP5: TestPoint, UTSVT_Special:TestPoint_HEX_3mmID
- removed U1: SHT45, Sensor_Humidity:Sensirion_DFN-4_1.5x1.5mm_P0.8mm_SHT4x_NoCentralPad
- removed U2: FS3000-1005, SamacSys_Parts:FS30001005
- removed U3: LMT87DCK, Package_TO_SOT_SMD:SOT-353_SC-70-5
- removed U4: Daughterboard Connector, UTSVT_Special:PeripheralSOM
Routing:
- net /CAN_L: track 51.1 -> 0.00 mm
- net /CAN_H: track 47.8 -> 0.00 mm
- net GNDA: track 26.3 -> 0.00 mm, vias 4 -> 0
- net /I2C1_SDA: track 23.4 -> 0.00 mm, vias 3 -> 0
- net /I2C1_SCL: track 22.6 -> 0.00 mm, vias 3 -> 0
- net /PA1(ADC): track 21.3 -> 0.00 mm, vias 2 -> 0
- net /I2C2_SCL: track 18.8 -> 0.00 mm, vias 3 -> 0
- net /I2C2_SDA: track 16.8 -> 0.00 mm, vias 3 -> 0
- net VDDA: track 16.3 -> 0.00 mm, vias 2 -> 0
- net /VDDA-out: track 9.41 -> 0.00 mm, vias 1 -> 0
- net +3.3V: track 6.04 -> 0.00 mm, vias 3 -> 0
- net GND: track 4.02 -> 0.00 mm, vias 8 -> 0
- net /3.3-out: track 3.13 -> 0.00 mm
- net +12V_In: track 2.54 -> 0.00 mm
- net /AFLW_TP1: track 2.31 -> 0.00 mm, vias 1 -> 0
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- removed copper zone on F.Cu, net +12V_In
- removed copper zone on F.Cu, net +3.3V
- removed copper zone on B.Cu, net GND
- removed copper zone on B.Cu, net GNDPWR
Other:
- board outline removed
- board text removed: "12V"
- board text removed: "3.3V"
- board text removed: "Airflow"
- board text removed: "Breakout"
- board text removed: "Data Acq Environment Board Ravi Shah 2024"
- board text removed: "GND"
- board text removed: "GNDPWR"
- board text removed: "Grid size is .25mm"
- board text removed: "Humidity"
- board text removed: "PSOM Connection"
- board text removed: "Temp"
- board text removed: "v1.0"

Commit message: not layout
Parts:
- added D1: 12V, LED_SMD:LED_0805_2012Metric, F.Cu at (206.2, 118.1)
- added D2: 3.3V, LED_SMD:LED_0805_2012Metric, F.Cu at (206.2, 121.1)
- added D3: PESD3V3L4BHCYL, PESD3V3L4BHCYL:SON45P80X130X43-6N, B.Cu at (163.7, 93.8)
- added F1: 250mA, Fuse:Fuse_1206_3216Metric, B.Cu at (158.5, 93.2)
- added J1: ENV, 1053091104:MOLEX_1053091104, F.Cu at (168.0, 97.2)
- added J2: CAN OUT, UTSVT_Connectors:Molex_MicroFit3.0_1x4xP3.00mm_PolarizingPeg_Vertical, F.Cu at (135.8, 124.8)
- added J3: CAN IN, UTSVT_Connectors:Molex_MicroFit3.0_1x4xP3.00mm_PolarizingPeg_Vertical, F.Cu at (156.5, 124.8)
- added LOGO2: Dr. Hallock, UTSVT_Special:Hallock_Image_Tiny, F.Cu at (207.5, 75.0)
- added LOGO3: UTSVT Logo, UTSVT_Special:UTSVT_Logo_Symbol, F.Cu at (208.0, 62.0)
- added LOGO4: Wolf, images:wolf, F.Cu at (209.5, 94.0)
- added R2: 5.1k, Resistor_SMD:R_0805_2012Metric, F.Cu at (210.6, 118.0)
- added R3: 680, Resistor_SMD:R_0805_2012Metric, F.Cu at (210.6, 121.0)
- added TP1: 12V, UTSVT_Special:TestPoint_HEX_3mmID, F.Cu at (201.5, 109.5)
- added TP2: GNDPWR, UTSVT_Special:TestPoint_HEX_3mmID, F.Cu at (205.5, 109.5)
- added TP4: 3.3V, UTSVT_Special:TestPoint_HEX_3mmID, F.Cu at (209.5, 109.5)
- added TP5: GND, UTSVT_Special:TestPoint_HEX_3mmID, F.Cu at (213.5, 109.5)
- added U4: Daughterboard Connector, UTSVT_Special:PeripheralSOM, F.Cu at (140.1, 89.3)

Commit message: layout finished
Parts:
- R2, R3: moved to B.Cu
- moved R2 59.4 mm to (164.3, 80.8)
- moved R3 58.8 mm to (164.3, 84.8)
- moved TP4 57.1 mm to (164.8, 74.0), turned to -90 degrees
- moved TP5 56.3 mm to (168.2, 76.0), turned to -90 degrees
- moved D1 53.0 mm to (168.5, 80.8), turned to 180 degrees
- moved D2 52.4 mm to (168.5, 84.8), turned to 180 degrees
- moved TP2 39.4 mm to (168.2, 122.2), turned to -90 degrees
- moved TP1 38.3 mm to (164.8, 120.2), turned to -90 degrees
- moved J1 1.25 mm to (166.8, 97.2)
- moved D3 1.22 mm to (163.5, 95.0), turned to 90 degrees
- moved J3 0.50 mm to (156.0, 124.8)
- moved J2 0.25 mm to (136.0, 124.8)
Routing:
- net /CAN_L: track 0.00 -> 61.7 mm, vias 0 -> 1
- net /CAN_H: track 0.00 -> 52.8 mm, vias 0 -> 2
- net GND: track 0.00 -> 26.1 mm, vias 0 -> 2
- net +3.3V: track 0.00 -> 23.7 mm, vias 0 -> 3
- net /I2C1_SCL: track 0.00 -> 11.6 mm
- net /I2C1_SDA: track 0.00 -> 10.3 mm, vias 0 -> 1
- net +12V: track 0.00 -> 2.73 mm, vias 0 -> 3
- net Net-(D2-A): track 0.00 -> 2.31 mm, vias 0 -> 1
- net Net-(D1-A): track 0.00 -> 2.31 mm, vias 0 -> 1
- net +3.3V_OUT: track 0.00 -> 1.45 mm
- added copper zone on B.Cu, net +12V
- added copper zone on B.Cu, net +3.3V
- added copper zone on B.Cu, net +3.3V_OUT
- added copper zone on F.Cu, net GND
- added copper zone on F.Cu, net GNDPWR
Other:
- board outline added: 53.2 x 62.8 mm
